Commit message: update models xacro

File: install/robot_description/share/robot_description/urdf/my_robot.urdf (robot description, URDF)
Before this commit: robot my_robot, 5 links, 4 joints
Links:
- added link arm_base_link, mass 0.5; collision box size=0.1 0.1 0.02; visual box size=0.1 0.1 0.02
- added link forearm_link, mass 0.3; collision cylinder length=0.3 radius=0.02; visual cylinder length=0.3 radius=0.02
- added link hand_link, mass 0.3; collision cylinder length=0.3 radius=0.02; visual cylinder length=0.3 radius=0.02
- link base_link: mass None -> 5.0; geometry collision box size=0.6 0.4 0.2; visual box size=0.6 0.4 0.2
- link caster_wheel_link: mass None -> 0.5; geometry collision sphere radius=0.05; visual sphere radius=0.05
- link left_wheel_link: mass None -> 1.0; geometry collision cylinder length=0.05 radius=0.1; visual cylinder length=0.05 radius=0.1
- link right_wheel_link: mass None -> 1.0; geometry collision cylinder length=0.05 radius=0.1; visual cylinder length=0.05 radius=0.1
Joints:
- added joint arm_base_forearm_joint: type revolute, parent arm_base_link, child forearm_link, origin xyz=0 0 0.02 rpy=0 0 0, axis 0 1 0, limit lower=0 upper=1.5707963267948966 effort=100 velocity=100
- added joint forearm_hand_joint: type revolute, parent forearm_link, child hand_link, origin xyz=0 0 0.3 rpy=0 0 0, axis 0 1 0, limit lower=0 upper=1.5707963267948966 effort=100 velocity=100
- added joint mobile_base_arm_joint: type fixed, parent base_link, child arm_base_link, origin xyz=0.15 0 0.2 rpy=0 0 0
- joint base_caster_wheel_joint: origin xyz=0.2 0 -0.05 rpy=0 0 0 -> xyz=0.19999999999999998 0 -0.05 rpy=0 0 0
