Commit message: box model

File: src/robot_description/urdf/rubot_mpuig2.urdf (robot description, URDF)
Before this commit: robot rubot, 9 links, 8 joints
Links:
- link base_link: geometry collision box size=0.26 0.15 0.1; visual box size=0.26 0.15 0.08
- link base_scan: geometry collision cylinder length=0.05 radius=0.05; visual cylinder length=0.05 radius=0.05
- link camera: geometry collision box size=0.05 0.05 0.025; visual box size=0.05 0.05 0.025
- link lower_left_wheel: geometry collision cylinder length=0.03 radius=0.05; visual cylinder length=0.03 radius=0.05
- link lower_right_wheel: geometry collision cylinder length=0.03 radius=0.05; visual cylinder length=0.03 radius=0.05
- link part: geometry collision box size=0.05 0.05 0.025; visual box size=0.05 0.05 0.025
- link upper_left_wheel: geometry collision cylinder length=0.03 radius=0.05; visual cylinder length=0.03 radius=0.05
- link upper_right_wheel: geometry collision cylinder length=0.03 radius=0.05; visual cylinder length=0.03 radius=0.05
Joints:
- joint base_link_joint: origin xyz=0 0 0 rpy=0 0 0 -> xyz=0 0 0.05 rpy=0 0 0
- joint joint_camera: origin xyz=0.120 0.0 0.09 rpy=0 0 0 -> xyz=0.130 0.0 0.05 rpy=0 0 0
- joint joint_part: origin xyz=-0.10 0.0 0.09 rpy=0 0 0 -> xyz=-0.10 0.0 0.08 rpy=0 0 0
- joint scan_joint: origin xyz=0 0 0.15 rpy=0 0 3.14 -> xyz=0 0 0.12 rpy=0 0 3.14
