Commit message: mecanum xacro model

File: src/my_robot_description/urdf/lidar.xacro (robot description, xacro)
@@ -1,8 +1,8 @@
 <?xml version="1.0"?>
 <robot xmlns:xacro="http://www.ros.org/wiki/xacro">
-    <xacro:property name="camera_length" value="0.01" />
+    <xacro:property name="camera_length" value="0.1" />
     <xacro:property name="camera_width" value="0.1" />
-    <xacro:property name="camera_height" value="0.05" />
-    <link name="camera_link">
+    <xacro:property name="camera_height" value="0.1" />
+    <link name="base_scan">
         <visual>
             <geometry>
@@ -19,28 +19,42 @@
                            xyz="0 0 0" rpy="0 0 0" />
     </link>
-    <joint name="base_camera_joint" type="fixed">
+    <joint name="base_scan_joint" type="fixed">
         <parent link="base_link" />
-        <child link="camera_link" />
-        <origin xyz="${(base_length + camera_length) / 2.0} 0 ${base_height / 2.0}" rpy="0 0 0" />
+        <child link="base_scan" />
+        <origin xyz="0 0 ${base_height+0.1}" rpy="0 0 0" />
     </joint>
-    <link name="camera_link_optical">
-    </link>
-    <joint name="camera_optical_joint" type="fixed">
-        <!-- these values have to be these values otherwise the gazebo camera
-            image won't be aligned properly with the frame it is supposedly
-            originating from -->
-        <origin xyz="0 0 0" rpy="${-pi/2} 0 ${-pi/2}"/>
-        <parent link="camera_link"/>
-        <child link="camera_link_optical"/>
-    </joint>
-    <gazebo reference="camera_link">
-        <material>Gazebo/Red</material>
-        <sensor name="camera_sensor" type="camera">
-            <pose>0 0 0 0 0 0</pose>
-            <visualize>true</visualize>
-            <update_rate>10.0</update_rate>
-            <plugin name="camera_controller" filename="libgazebo_ros_camera.so">
-                <frame_name>camera_link_optical</frame_name>
-            </plugin>
+    <gazebo reference="base_scan">
+        <sensor name="lidar" type="ray">
+        <pose>0.215 0 0.215 0 0 0</pose>
+        <always_on>true</always_on>
+        <visualize>false</visualize>
+        <update_rate>5</update_rate>
+        <ray>
+            <scan>
+                <horizontal>
+                    <samples>720</samples>
+                    <resolution>1.00000</resolution>
+                    <min_angle>0.000000</min_angle>
+                    <max_angle>6.280000</max_angle>
+                </horizontal>
+            </scan>
+            <range>
+                <min>0.120000</min>
+                <max>3.5</max>
+                <resolution>0.015000</resolution>
+            </range>
+            <noise>
+                <type>gaussian</type>
+                <mean>0.0</mean>
+                <stddev>0.01</stddev>
+            </noise>
+        </ray>
+        <plugin name="scan" filename="libgazebo_ros_ray_sensor.so">
+            <ros>
+                <remapping>~/out:=scan</remapping>
+            </ros>
+            <output_type>sensor_msgs/LaserScan</output_type>
+            <frame_name>base_scan</frame_name>
+        </plugin>
         </sensor>
     </gazebo>

File: src/my_robot_description/urdf/mecanum_base_gazebo.xacro (robot description, xacro)
@@ -4,32 +4,33 @@
         <material>Gazebo/Blue</material>
     </gazebo>
-    <gazebo reference="right_wheel_link">
+    <gazebo reference="lower_right_wheel_link">
         <material>Gazebo/Grey</material>
     </gazebo>
-    <gazebo reference="left_wheel_link">
+    <gazebo reference="lower_left_wheel_link">
         <material>Gazebo/Grey</material>
     </gazebo>
-    <gazebo reference="caster_wheel_link">
+    <gazebo reference="upper_right_wheel_link">
         <material>Gazebo/Grey</material>
-        <mu1 value="0.1" />
-        <mu2 value="0.1" />
+    </gazebo>
+    <gazebo reference="upper_left_wheel_link">
+        <material>Gazebo/Grey</material>
     </gazebo>
     <gazebo>
-        <plugin name="diff_drive_controller" filename="libgazebo_ros_diff_drive.so">
-            <!-- Update rate in Hz -->
-            <update_rate>50</update_rate>
-            <!-- wheels -->
-            <left_joint>base_left_wheel_joint</left_joint>
-            <right_joint>base_right_wheel_joint</right_joint>
-            <!-- kinematics -->
-            <wheel_separation>0.45</wheel_separation>
-            <wheel_diameter>0.2</wheel_diameter>
-            <!-- output -->
-            <publish_odom>true</publish_odom>
-            <publish_odom_tf>true</publish_odom_tf>
-            <publish_wheel_tf>true</publish_wheel_tf>
-            <odometry_topic>odom</odometry_topic>
-            <odometry_frame>odom</odometry_frame>
-            <robot_base_frame>base_footprint</robot_base_frame>
+        <plugin name="mecanum_controller" filename="libgazebo_ros_omni_drive.so">
+            <commandTopic>cmd_vel</commandTopic>
+            <odometryTopic>odom</odometryTopic>
+            <odometryFrame>odom</odometryFrame>
+            <odometryRate>20.0</odometryRate>
+            <robotBaseFrame>base_footprint</robotBaseFrame>
+            <wheel_radius>0.04</wheel_radius>
+            <base_length>0.65</base_length>
+            <base_width>0.65</base_width>
+            <front_left_joint>upper_left_wheel_joint</front_left_joint>
+            <front_right_joint>upper_right_wheel_joint</front_right_joint>
+            <rear_left_joint>lower_left_wheel_joint</rear_left_joint>
+            <rear_right_joint>lower_right_wheel_joint</rear_right_joint>
+            <wheel_max_speed> 20.0 </wheel_max_speed>
+            <wheel_acceleration> 10.0</wheel_acceleration>
+            <joint_config>1 1 1 1</joint_config>
         </plugin>
     </gazebo>

File: src/my_robot_description/urdf/mecanum_mobile_base.xacro (robot description, xacro)
@@ -43,23 +43,8 @@
         </link>
     </xacro:macro>
-    <xacro:wheel_link prefix="right" />
-    <xacro:wheel_link prefix="left" />
-    <link name="caster_wheel_link">
-        <visual>
-            <geometry>
-                <sphere radius="${wheel_radius / 2.0}" />
-            </geometry>
-            <origin xyz="0 0 0" rpy="0 0 0" />
-            <material name="grey" />
-        </visual>
-        <collision>
-            <geometry>
-                <sphere radius="${wheel_radius / 2.0}" />
-            </geometry>
-            <origin xyz="0 0 0" rpy="0 0 0" />
-        </collision>
-        <xacro:sphere_inertia m="0.5" r="${2*wheel_radius / 2.0}"
-                              xyz="0 0 0" rpy="0 0 0" />
-    </link>
+    <xacro:wheel_link prefix="lower_right" />
+    <xacro:wheel_link prefix="lower_left" />
+    <xacro:wheel_link prefix="upper_right" />
+    <xacro:wheel_link prefix="upper_left" />
     <joint name="base_joint" type="fixed">
         <parent link="base_footprint" />
@@ -67,20 +52,27 @@
         <origin xyz="0 0 ${wheel_radius}" rpy="0 0 0"/>
     </joint>
-    <joint name="base_right_wheel_joint" type="continuous">
+    <joint name="lower_right_wheel_joint" type="continuous">
         <parent link="base_link" />
-        <child link="right_wheel_link" />
+        <child link="lower_right_wheel_link" />
         <origin xyz="${-base_length / 4.0} ${-(base_width + wheel_length) / 2.0} 0" rpy="0 0 0" />
         <axis xyz="0 1 0" />
     </joint>
-    <joint name="base_left_wheel_joint" type="continuous">
+    <joint name="lower_left_wheel_joint" type="continuous">
         <parent link="base_link" />
-        <child link="left_wheel_link" />
+        <child link="lower_left_wheel_link" />
         <origin xyz="${-base_length / 4.0} ${(base_width + wheel_length) / 2.0} 0" rpy="0 0 0" />
         <axis xyz="0 1 0" />
     </joint>
-    <joint name="base_caster_wheel_joint" type="fixed">
+    <joint name="upper_right_wheel_joint" type="continuous">
         <parent link="base_link" />
-        <child link="caster_wheel_link" />
-        <origin xyz="${base_length / 3.0} 0 ${-wheel_radius / 2.0}" rpy="0 0 0" />
+        <child link="upper_right_wheel_link" />
+        <origin xyz="${base_length / 4.0} ${-(base_width + wheel_length) / 2.0} 0" rpy="0 0 0" />
+        <axis xyz="0 1 0" />
+    </joint>
+    <joint name="upper_left_wheel_joint" type="continuous">
+        <parent link="base_link" />
+        <child link="upper_left_wheel_link" />
+        <origin xyz="${base_length / 4.0} ${(base_width + wheel_length) / 2.0} 0" rpy="0 0 0" />
+        <axis xyz="0 1 0" />
     </joint>
 </robot>

File: src/my_robot_description/urdf/my_mecanum_robot.urdf.xacro (robot description, xacro)
@@ -2,6 +2,6 @@
 <robot name="my_robot" xmlns:xacro="http://www.ros.org/wiki/xacro">
     <xacro:include filename="common_properties.xacro" />
-    <xacro:include filename="mobile_base.xacro" />
-    <xacro:include filename="mobile_base_gazebo.xacro" />
+    <xacro:include filename="mecanum_mobile_base.xacro" />
+    <xacro:include filename="mecanum_base_gazebo.xacro" />
     <xacro:include filename="arm.xacro" />
     <xacro:include filename="arm_gazebo.xacro" />
@@ -13,4 +13,3 @@
         <origin xyz="${base_length / 4.0} 0 ${base_height}" rpy="0 0 0" />
     </joint>
-    <!-- <xacro:include filename="camera.xacro" /> -->
 </robot>

Commit message: mecanum scalled model

File: src/my_robot_description/urdf/lidar.xacro (robot description, xacro)
@@ -1,11 +1,10 @@
 <?xml version="1.0"?>
 <robot xmlns:xacro="http://www.ros.org/wiki/xacro">
-    <xacro:property name="camera_length" value="0.1" />
-    <xacro:property name="camera_width" value="0.1" />
-    <xacro:property name="camera_height" value="0.1" />
+    <xacro:property name="lidar_radius" value="0.05" />
+    <xacro:property name="lidar_length" value="0.02" />
     <link name="base_scan">
         <visual>
             <geometry>
-                <box size="${camera_length} ${camera_width} ${camera_height}" />
+                <cylinder radius="${lidar_radius}" length="${lidar_length}" />
             </geometry>
             <material name="grey" />
@@ -13,14 +12,14 @@
         <collision>
             <geometry>
-                <box size="${camera_length} ${camera_width} ${camera_height}" />
+                <cylinder radius="${lidar_radius}" length="${lidar_length}" />
             </geometry>
         </collision>
-        <xacro:box_inertia m="0.1" l="${camera_length}" w="${camera_width}" h="${camera_height}"
-                           xyz="0 0 0" rpy="0 0 0" />
+        <xacro:cylinder_inertia m="0.1" r="${2*lidar_radius}" h="${2*lidar_length}"
+                                xyz="0 0 0" rpy="0 0 0" />
     </link>
     <joint name="base_scan_joint" type="fixed">
         <parent link="base_link" />
         <child link="base_scan" />
-        <origin xyz="0 0 ${base_height+0.1}" rpy="0 0 0" />
+        <origin xyz="0 0 ${base_height+0.05}" rpy="0 0 0" />
     </joint>
     <gazebo reference="base_scan">

File: src/my_robot_description/urdf/mecanum_mobile_base.xacro (robot description, xacro)
@@ -1,9 +1,9 @@
 <?xml version="1.0"?>
 <robot xmlns:xacro="http://www.ros.org/wiki/xacro">
-    <xacro:property name="base_length" value="0.6" />
-    <xacro:property name="base_width" value="0.4" />
-    <xacro:property name="base_height" value="0.2" />
-    <xacro:property name="wheel_radius" value="0.1" />
-    <xacro:property name="wheel_length" value="0.05" />
+    <xacro:property name="base_length" value="0.26" />
+    <xacro:property name="base_width" value="0.15" />
+    <xacro:property name="base_height" value="0.08" />
+    <xacro:property name="wheel_radius" value="0.04" />
+    <xacro:property name="wheel_length" value="0.01" />
     <link name="base_footprint" />
     <!-- collision and inertia box close to floor for lateral movements -->
@@ -14,5 +14,5 @@
             </geometry>
             <origin xyz="0 0 ${base_height / 2.0}" rpy="0 0 0" />
-            <material name="blue" />
+            <material name="yellow" />
         </visual>
         <collision>

File: src/my_robot_description/urdf/mecanum_mobile_base_gazebo.xacro (robot description, xacro)
@@ -3,5 +3,5 @@
     <!-- low friction with base and high friction with wheels -->
     <gazebo reference="base_link">
-        <material>Gazebo/Blue</material>
+        <material>Gazebo/Yellow</material>
         <mu1>0.005</mu1>
         <mu2>0.005</mu2>

File: src/my_robot_description/urdf/my_mecanum_robot.urdf.xacro (robot description, xacro)
@@ -4,6 +4,6 @@
     <xacro:include filename="mecanum_mobile_base.xacro" />
     <xacro:include filename="mecanum_mobile_base_gazebo.xacro" />
-    <xacro:include filename="arm.xacro" />
-    <xacro:include filename="arm_gazebo.xacro" />
+    <xacro:include filename="mecanum_arm.xacro" />
+    <xacro:include filename="mecanum_arm_gazebo.xacro" />
     <xacro:include filename="camera.xacro" />
     <xacro:include filename="lidar.xacro" />

Commit message: selfnav

File: src/my_robot_description/urdf/lidar.xacro (robot description, xacro)
@@ -21,5 +21,5 @@
         <parent link="base_link" />
         <child link="base_scan" />
-        <origin xyz="0 0 ${base_height+0.05}" rpy="0 0 0" />
+        <origin xyz="0 0 ${base_height+0.05}" rpy="0 0 3.14" />
     </joint>
     <gazebo reference="base_scan">
