Commit message: mu and pid adjustments

File: src/my_robot_description/urdf/mecanum_mobile_base.xacro (robot description, xacro)
@@ -7,4 +7,5 @@
     <xacro:property name="wheel_length" value="0.05" />
     <link name="base_footprint" />
+    <!-- collision and inertia box close to floor for lateral movements -->
     <link name="base_link">
         <visual>
@@ -19,8 +20,8 @@
                 <box size="${base_length} ${base_width} ${base_height}" />
             </geometry>
-            <origin xyz="0 0 ${base_height / 2.0}" rpy="0 0 0" />
+            <origin xyz="0 0 0" rpy="0 0 0" />
         </collision>
         <xacro:box_inertia m="5.0" l="${2*base_length}" w="${2*base_width}" h="${2*base_height}"
-                           xyz="0 0 ${base_height / 2.0}" rpy="0 0 0" />
+                           xyz="0 0 0" rpy="0 0 0" />
     </link>
     <xacro:macro name="wheel_link" params="prefix">

File: src/my_robot_description/urdf/mecanum_mobile_base_gazebo.xacro (robot description, xacro)
@@ -1,26 +1,53 @@
 <?xml version="1.0"?>
 <robot xmlns:xacro="http://www.ros.org/wiki/xacro">
+    <!-- low friction with base and high friction with wheels -->
     <gazebo reference="base_link">
         <material>Gazebo/Blue</material>
+        <mu1>0.005</mu1>
+        <mu2>0.005</mu2>
     </gazebo>
     <gazebo reference="lower_right_wheel_link">
         <material>Gazebo/Grey</material>
-        <mu1>0.5</mu1>
-        <mu2>0.5</mu2>
+        <mu1>0.4</mu1>
+        <mu2>0.4</mu2>
+        <kp>1000</kp>
+        <ki>100</ki>
+        <kd>1</kd>
+        <minDepth>0.001</minDepth>
+        <maxVel>0.5</maxVel>
+        <fdir1>1 0 0</fdir1>
     </gazebo>
     <gazebo reference="lower_left_wheel_link">
         <material>Gazebo/Grey</material>
-        <mu1>0.5</mu1>
-        <mu2>0.5</mu2>
+        <mu1>0.4</mu1>
+        <mu2>0.4</mu2>
+        <kp>1000</kp>
+        <ki>100</ki>
+        <kd>1</kd>
+        <minDepth>0.001</minDepth>
+        <maxVel>0.5</maxVel>
+        <fdir1>1 0 0</fdir1>
     </gazebo>
     <gazebo reference="upper_right_wheel_link">
         <material>Gazebo/Grey</material>
-        <mu1>0.5</mu1>
-        <mu2>0.5</mu2>
+        <mu1>0.4</mu1>
+        <mu2>0.4</mu2>
+        <kp>1000</kp>
+        <ki>100</ki>
+        <kd>1</kd>
+        <minDepth>0.001</minDepth>
+        <maxVel>0.5</maxVel>
+        <fdir1>1 0 0</fdir1>
     </gazebo>
     <gazebo reference="upper_left_wheel_link">
         <material>Gazebo/Grey</material>
-        <mu1>0.5</mu1>
-        <mu2>0.5</mu2>
+        <mu1>0.4</mu1>
+        <mu2>0.4</mu2>
+        <kp>1000</kp>
+        <ki>100</ki>
+        <kd>1</kd>
+        <minDepth>0.001</minDepth>
+        <maxVel>0.5</maxVel>
+        <fdir1>1 0 0</fdir1>
     </gazebo>
     <gazebo>
@@ -32,12 +59,12 @@
             <robotBaseFrame>base_footprint</robotBaseFrame>
             <wheel_radius>0.04</wheel_radius>
-            <base_length>0.65</base_length>
-            <base_width>0.65</base_width>
+            <base_length>0.26</base_length>
+            <base_width>0.15</base_width>
             <front_left_joint>upper_left_wheel_joint</front_left_joint>
             <front_right_joint>upper_right_wheel_joint</front_right_joint>
             <rear_left_joint>lower_left_wheel_joint</rear_left_joint>
             <rear_right_joint>lower_right_wheel_joint</rear_right_joint>
-            <wheel_max_speed> 20.0 </wheel_max_speed>
-            <wheel_acceleration> 10.0</wheel_acceleration>
+            <wheel_max_speed> 2.0 </wheel_max_speed>
+            <wheel_acceleration> 1.0</wheel_acceleration>
             <joint_config>1 1 1 1</joint_config>
         </plugin>

Commit message: navigation1

File: src/my_robot_description/urdf/mecanum_mobile_base.xacro (robot description, xacro)
@@ -30,4 +30,5 @@
                 <geometry>
                     <cylinder radius="${wheel_radius}" length="${wheel_length}" />
+                    <!--<mesh filename="package://my_robot_description/meshes/left_tire.stl" scale="0.001 0.001 0.001"/>-->
                 </geometry>
                 <origin xyz="0 0 0" rpy="${pi / 2.0} 0 0" />

File: src/my_robot_description/urdf/mecanum_mobile_base_gazebo.xacro (robot description, xacro)
@@ -11,10 +11,10 @@
         <mu1>0.4</mu1>
         <mu2>0.4</mu2>
-        <kp>1000</kp>
+        <!--<kp>1000</kp>
         <ki>100</ki>
         <kd>1</kd>
         <minDepth>0.001</minDepth>
         <maxVel>0.5</maxVel>
-        <fdir1>1 0 0</fdir1>
+        <fdir1>1 0 0</fdir1>-->
     </gazebo>
     <gazebo reference="lower_left_wheel_link">
@@ -22,10 +22,10 @@
         <mu1>0.4</mu1>
         <mu2>0.4</mu2>
-        <kp>1000</kp>
+        <!--<kp>1000</kp>
         <ki>100</ki>
         <kd>1</kd>
         <minDepth>0.001</minDepth>
         <maxVel>0.5</maxVel>
-        <fdir1>1 0 0</fdir1>
+        <fdir1>1 0 0</fdir1>-->
     </gazebo>
     <gazebo reference="upper_right_wheel_link">
@@ -33,10 +33,10 @@
         <mu1>0.4</mu1>
         <mu2>0.4</mu2>
-        <kp>1000</kp>
+        <!--<kp>1000</kp>
         <ki>100</ki>
         <kd>1</kd>
         <minDepth>0.001</minDepth>
         <maxVel>0.5</maxVel>
-        <fdir1>1 0 0</fdir1>
+        <fdir1>1 0 0</fdir1>-->
     </gazebo>
     <gazebo reference="upper_left_wheel_link">
@@ -44,10 +44,10 @@
         <mu1>0.4</mu1>
         <mu2>0.4</mu2>
-        <kp>1000</kp>
+        <!--<kp>1000</kp>
         <ki>100</ki>
         <kd>1</kd>
         <minDepth>0.001</minDepth>
         <maxVel>0.5</maxVel>
-        <fdir1>1 0 0</fdir1>
+        <fdir1>1 0 0</fdir1>-->
     </gazebo>
     <gazebo>
