Commit message: inertia movement

File: src/my_robot_description/urdf/mecanum_arm.xacro (robot description, xacro)
@@ -22,5 +22,5 @@
             <origin xyz="0 0 ${arm_base_height / 2.0}" rpy="0 0 0" />
         </collision>
-        <xacro:box_inertia m="0.5" l="${2*arm_base_length}" w="${2*arm_base_width}" h="${2*arm_base_height}"
+        <xacro:box_inertia m="0.1" l="${2*arm_base_length}" w="${2*arm_base_width}" h="${2*arm_base_height}"
                            xyz="0 0 ${arm_base_height / 2.0}" rpy="0 0 0" />
     </link>
@@ -39,5 +39,5 @@
             <origin xyz="0 0 ${forearm_length / 2.0}" rpy="0 0 0" />
         </collision>
-        <xacro:cylinder_inertia m="0.3" r="${2*forearm_radius}" h="${2*forearm_length}"
+        <xacro:cylinder_inertia m="0.1" r="${2*forearm_radius}" h="${2*forearm_length}"
                                 xyz="0 0 ${forearm_length / 2.0}" rpy="0 0 0" />
     </link>
@@ -56,5 +56,5 @@
             <origin xyz="0 0 ${hand_length / 2.0}" rpy="0 0 0" />
         </collision>
-        <xacro:cylinder_inertia m="0.3" r="${2*hand_radius}" h="${2*hand_length}"
+        <xacro:cylinder_inertia m="0.1" r="${2*hand_radius}" h="${2*hand_length}"
                                 xyz="0 0 ${hand_length / 2.0}" rpy="0 0 0" />
     </link>

File: src/my_robot_description/urdf/mecanum_mobile_base.xacro (robot description, xacro)
@@ -5,5 +5,5 @@
     <xacro:property name="base_height" value="0.08" />
     <xacro:property name="wheel_radius" value="0.04" />
-    <xacro:property name="wheel_length" value="0.01" />
+    <xacro:property name="wheel_length" value="0.02" />
     <link name="base_footprint" />
     <!-- collision and inertia box close to floor for lateral movements -->
@@ -20,8 +20,8 @@
                 <box size="${base_length} ${base_width} ${base_height}" />
             </geometry>
-            <origin xyz="0 0 0" rpy="0 0 0" />
+            <origin xyz="0 0 0.0" rpy="0 0 0" />
         </collision>
-        <xacro:box_inertia m="5.0" l="${2*base_length}" w="${2*base_width}" h="${2*base_height}"
-                           xyz="0 0 0" rpy="0 0 0" />
+        <xacro:box_inertia m="4.0" l="${2*base_length}" w="${2*base_width}" h="${2*base_height}"
+                           xyz="0 0 0.0" rpy="0 0 0" />
     </link>
     <xacro:macro name="wheel_link" params="prefix">
@@ -41,5 +41,5 @@
                 <origin xyz="0 0 0" rpy="${pi / 2.0} 0 0" />
             </collision>
-            <xacro:cylinder_inertia m="1.0" r="${2*wheel_radius}" h="${2*wheel_length}"
+            <xacro:cylinder_inertia m="0.2" r="${2*wheel_radius}" h="${2*wheel_length}"
                                     xyz="0 0 0" rpy="${pi / 2.0} 0 0" />
         </link>

File: src/my_robot_description/urdf/mecanum_mobile_base_gazebo.xacro (robot description, xacro)
@@ -10,5 +10,5 @@
         <material>Gazebo/Grey</material>
         <mu1>0.4</mu1>
-        <mu2>0.4</mu2>
+        <mu2>0.2</mu2>
         <!--<kp>1000</kp>
         <ki>100</ki>
@@ -21,5 +21,5 @@
         <material>Gazebo/Grey</material>
         <mu1>0.4</mu1>
-        <mu2>0.4</mu2>
+        <mu2>0.2</mu2>
         <!--<kp>1000</kp>
         <ki>100</ki>
@@ -32,5 +32,5 @@
         <material>Gazebo/Grey</material>
         <mu1>0.4</mu1>
-        <mu2>0.4</mu2>
+        <mu2>0.2</mu2>
         <!--<kp>1000</kp>
         <ki>100</ki>
@@ -43,5 +43,5 @@
         <material>Gazebo/Grey</material>
         <mu1>0.4</mu1>
-        <mu2>0.4</mu2>
+        <mu2>0.2</mu2>
         <!--<kp>1000</kp>
         <ki>100</ki>
