Commit message: stl files

File: src/my_robot_description/urdf/rubot_mpuig.urdf (robot description, URDF)
Before this commit: robot rubot, 9 links, 8 joints
Links:
- link base_link: geometry collision box size=0.23 0.12 0.1; visual mesh filename=file://$(find my_robot_description)/meshes/base_link.stl scale=0.001 0.001 0.001
- link base_scan: geometry collision cylinder length=0.05 radius=0.05; visual mesh filename=file://$(find my_robot_description)/meshes/Lidar.stl scale=0.001 0.001 0.001
- link lower_left_wheel: geometry collision cylinder length=0.03 radius=0.055; visual mesh filename=file://$(find my_robot_description)/meshes/lower_left_wheel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 scale=0.001 0.001 0.001
- link lower_right_wheel: geometry collision cylinder length=0.03 radius=0.055; visual mesh filename=file://$(find my_robot_description)/meshes/lower_right_whee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 scale=0.001 0.001 0.001
- link part: geometry collision box size=0.05 0.05 0.025; visual mesh filename=file://$(find my_robot_description)/meshes/number2.stl scale=0.0008 0.0008 0.0008
- link upper_left_wheel: geometry collision cylinder length=0.03 radius=0.055; visual mesh filename=file://$(find my_robot_description)/meshes/upper_left_wheel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 scale=0.001 0.001 0.001
- link upper_right_wheel: geometry collision cylinder length=0.03 radius=0.055; visual mesh filename=file://$(find my_robot_description)/meshes/upper_right_whee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 scale=0.001 0.001 0.001
Joints:
- joint base_link_joint: origin xyz=0 0 0.05 rpy=0 0 0 -> xyz=0 0 0 rpy=0 0 0
- joint scan_joint: origin xyz=0 0 0.12 rpy=0 0 3.14 -> xyz=0 0 0.14 rpy=0 0 3.14
