Commit message: bringup mecanum

File: src/my_robot_description/urdf/rubot/rubot_mecanum.urdf (robot description, URDF)
Before this commit: robot rubot, 9 links, 8 joints
Links:
- link base_link: geometry collision box size=0.23 0.12 0.1; visual mesh filename=file://$(find my_robot_description)/meshes/rubot/base_link.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 scale=0.001 0.001 0.001
- link base_scan: geometry collision cylinder length=0.05 radius=0.05; visual mesh filename=file://$(find my_robot_description)/meshes/rubot/Lidar.stl scale=0.001 0.001 0.001
- link lower_left_wheel: geometry collision cylinder length=0.03 radius=0.055; visual mesh filename=file://$(find my_robot_description)/meshes/rubot/lower_left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 scale=0.001 0.001 0.001
- link lower_right_wheel: geometry collision cylinder length=0.03 radius=0.055; visual mesh filename=file://$(find my_robot_description)/meshes/rubot/lower_righ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 scale=0.001 0.001 0.001
- link part: geometry collision box size=0.05 0.05 0.025; visual mesh filename=file://$(find my_robot_description)/meshes/rubot/number2.stl scale=0.0008 0.0008 0.0008
- link upper_left_wheel: geometry collision cylinder length=0.03 radius=0.055; visual mesh filename=file://$(find my_robot_description)/meshes/rubot/upper_left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 scale=0.001 0.001 0.001
- link upper_right_wheel: geometry collision cylinder length=0.03 radius=0.055; visual mesh filename=file://$(find my_robot_description)/meshes/rubot/upper_righ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 scale=0.001 0.001 0.001
