Commit message: ...

File: src/my_robot_description/urdf/rubot/rubot_custom.urdf (robot description, URDF)
Before this commit: robot rubot, 10 links, 9 joints
Links:
- removed link part
- link top_part: geometry collision box size=0.1 0.1 0.05; visual mesh filename=file://$(find my_robot_description)/meshes/rubot/bin_arc.stl scale=0.005 0.005 0.005
Joints:
- removed joint joint_part
- joint top_part_joint: origin xyz=0 0 0.1 rpy=0 0 0 -> xyz=0 0 0 rpy=0 0 0

Commit message: created custom robot and world

File: src/my_robot_description/urdf/rubot/rubot_custom.urdf (robot description, URDF)
Before this commit: robot rubot, 9 links, 8 joints
Links:
- link top_part: geometry collision box size=0.1 0.1 0.05; visual mesh filename=file://$(find my_robot_description)/meshes/rubot/bin_arc.stl scale=0.003 0.003 0.003
