Commit message: limo model urdf

File: src/my_robot_description/urdf/limo/rubot_limo.urdf (robot description, URDF)
Before this commit: robot limo, 9 links, 8 joints
Links:
- link base_link: geometry collision box size=0.23 0.12 0.1; visual mesh filename=file://$(find my_robot_description)/meshes/limo/limo.stl scale=0.001 0.001 0.001
- link base_scan: geometry collision cylinder length=0.015 radius=0.03; visual cylinder length=0.015 radius=0.03
- link camera: geometry collision box size=0.02 0.05 0.025; visual box size=0.02 0.05 0.025
- link part: geometry collision box size=0.05 0.05 0.025; visual box size=0.05 0.05 0.010
Joints:
- joint joint_camera: origin xyz=0.130 0.0 0.05 rpy=0 0 0 -> xyz=0.085 0.0 0.18 rpy=0 0 0
- joint joint_part: origin xyz=-0.10 0.0 0.08 rpy=0 0 0 -> xyz=-0.05 0.0 0.15 rpy=0 0 0
- joint lower_left_wheel_joint: origin xyz=-0.085 0.1 0 rpy=0 0 0 -> xyz=-0.085 0.06 0.02 rpy=0 0 0
- joint lower_right_wheel_joint: origin xyz=-0.085 -0.1 0 rpy=0 0 3.14 -> xyz=-0.085 -0.06 0.02 rpy=0 0 3.14
- joint scan_joint: origin xyz=0 0 0.14 rpy=0 0 3.14 -> xyz=0.11 0 0.12 rpy=0 0 3.14
- joint upper_left_wheel_joint: origin xyz=0.07 0.1 0 rpy=0 0 0 -> xyz=0.07 0.06 0.02 rpy=0 0 0
- joint upper_right_wheel_joint: origin xyz=0.07 -0.1 0 rpy=0 0 3.14 -> xyz=0.07 -0.06 0.02 rpy=0 0 3.14

Commit message: updated slam turtlebot3

File: src/my_robot_description/urdf/limo/rubot_limo.urdf (robot description, URDF)
Before this commit: robot limo, 9 links, 8 joints
Joints:
- joint scan_joint: origin xyz=0.11 0 0.12 rpy=0 0 3.14 -> xyz=0.11 0 0.12 rpy=0 0 0
